Commit message: update

File: robot_models/left_leg/left_leg.urdf (robot description, URDF)
Before this commit: robot left_leg, 7 links, 6 joints
Joints:
- removed joint Left_Ankle_Pitch
- removed joint Left_Ankle_Roll
- removed joint Left_Hip_Pitch
- removed joint Left_Hip_Roll
- removed joint Left_Hip_Yaw
- removed joint Left_Knee
- added joint left_ankle_pitch: type revolute, parent Left_Ankle_Roll_1, child Left_Foot_1, origin xyz=-0.019 -0.015 0.0 rpy=0 0 0, axis -0.0 1.0 -0.0, limit lower=-0.52 upper=0.5 effort=100 velocity=10
- added joint left_ankle_roll: type revolute, parent Left_Shank_1, child Left_Ankle_Roll_1, origin xyz=0.019 -0.017 -0.335 rpy=0 0 0, axis -1.0 -0.0 0.0, limit lower=-0.349 upper=0.349 effort=12 velocity=10
- added joint left_hip_pitch: type revolute, parent world, child Left_Hip_Pitch_1, origin xyz=0.0 0.089761 -0.081437 rpy=0 0 0, axis -0.0 0.965926 -0.258819, limit lower=-1.57 upper=1.57 effort=48 velocity=10
- added joint left_hip_roll: type revolute, parent Left_Hip_Pitch_1, child Left_Link2_Hip_1, origin xyz=0.0445 0.072444 -0.019412 rpy=0 0 0, axis 1.0 0.0 -0.0, limit lower=-0.785 upper=0.785 effort=48 velocity=10
- added joint left_hip_yaw: type revolute, parent Left_Link2_Hip_1, child Left_Thigh_1, origin xyz=-0.0445 0.0 -0.1205 rpy=0 0 0, axis -0.0 0.0 -1.0, limit lower=-0.785 upper=0.785 effort=100 velocity=10
- added joint left_knee: type revolute, parent Left_Thigh_1, child Left_Shank_1, origin xyz=0.0 0.017 -0.2035 rpy=0 0 0, axis -0.0 1.0 0.0, limit lower=0 upper=2.094 effort=100 velocity=10

Commit message: test base param and regressor calculation by compare to pin inverse dynamic RNEA

File: robot_models/left_leg/left_leg.urdf (robot description, URDF)
Before this commit: robot left_leg, 7 links, 6 joints
Joints:
- joint left_ankle_pitch: limit lower=-0.52 upper=0.5 effort=100 velocity=10 -> lower=-1.57 upper=1.57 effort=48 velocity=10
- joint left_ankle_roll: limit lower=-0.349 upper=0.349 effort=12 velocity=10 -> lower=-1.57 upper=1.57 effort=48 velocity=10
- joint left_hip_roll: limit lower=-0.785 upper=0.785 effort=48 velocity=10 -> lower=-1.57 upper=1.57 effort=48 velocity=10
- joint left_hip_yaw: limit lower=-0.785 upper=0.785 effort=100 velocity=10 -> lower=-1.57 upper=1.57 effort=48 velocity=10
- joint left_knee: limit lower=0 upper=2.094 effort=100 velocity=10 -> lower=-1.57 upper=1.57 effort=48 velocity=10

Commit message: add mujoco inverse dyna, remove collision geom in urdf

File: robot_models/left_leg/left_leg.urdf (robot description, URDF)
Before this commit: robot left_leg, 7 links, 6 joints
Links:
- link Left_Ankle_Roll_1: geometry visual mesh filename=meshes/Left_Ankle_Roll_1.stl scale=0.001 0.001 0.001
- link Left_Foot_1: geometry visual mesh filename=meshes/Left_Foot_1.stl scale=0.001 0.001 0.001
- link Left_Hip_Pitch_1: geometry visual mesh filename=meshes/Left_Hip_Pitch_1.stl scale=0.001 0.001 0.001
- link Left_Link2_Hip_1: geometry visual mesh filename=meshes/Left_Link2_Hip_1.stl scale=0.001 0.001 0.001
- link Left_Shank_1: geometry visual mesh filename=meshes/Left_Shank_1.stl scale=0.001 0.001 0.001
- link Left_Thigh_1: geometry visual mesh filename=meshes/Left_Thigh_1.stl scale=0.001 0.001 0.001

Commit message: add mjc sysid check

File: robot_models/left_leg/left_leg.urdf (robot description, URDF)
Before this commit: robot left_leg, 7 links, 6 joints
Joints:
- joint left_hip_pitch: axis -0.0 0.965926 -0.258819 -> 0 1 0
